File: RCDongle.brd (EAGLE design)
At the start: 100 x 80 mm, 21 parts, among them IC1 AT90USB162A, Q1 8MHz

Commit message: Update RCDongle.brd
Parts:
- C5, C6: value 15pF -> 18pF
- D1: device rcdongle:P-PRTR5V0U2X -> dn-electronics:P-SOT143BE
- IC1: value AT90USB162A -> AT90USB162; device adafruit:TQFP32-08 -> dn-electronics:P-TQFP32
- IR1: value (none) -> TSOP35; device rcdongle:P-TSOP35 -> dn-electronics:P-TSOP35
- JP1: device rcdongle:P-HWBRST -> dn-electronics:P-1X03
- JP2: device rcdongle:P-1X03 -> dn-electronics:P-1X03
- SW1, SW2: device rcdongle:P-SMTSWITCH -> dn-electronics:P-SWITCH-SMT-DTSM31NV
- U1: device rcdongle:P-USBAPLUG-V1 -> dn-electronics:P-USB-TYPEA-PLUG
- moved JP1 22.7 mm to (63.2, 41.3), turned to 90 degrees
- moved JP2 22.7 mm to (43.8, 29.5), turned to 270 degrees
- moved IR1 1.43 mm to (36.6, 21.1)
Connections:
- net GND: now also JP2.3; no longer JP1.3
- net N$11: now also JP2.1; no longer JP1.1
- net N$12: now also JP1.3; no longer JP2.3
- net N$5: now also JP1.1; no longer JP2.1
- net N$6: now also JP1.2; no longer JP2.2
- net N$9: now also JP2.2; no longer JP1.2
