File: RCDongle.sch (EAGLE design)
At the start: 21 parts, among them IC1 AT90USB162A, Q1 8MHz

Commit message: Update RCDongle.sch
Parts:
- C5, C6: value 15pF -> 18pF
- D1: device david-norman:PRTR5V0U2X -> dn-electronics:PRTR5V0U2X
- IC1: value AT90USB162A -> AT90USB162; device adafruit:AT90USB162A -> dn-electronics:AT90USB162
- IR1: value (none) -> TSOP35; device david-norman:TSOP35 -> dn-electronics:TSOP35
- JP1: device david-norman:AVR-USB-HWB/RST -> dn-electronics:HEADER-1X03
- JP2: device david-norman:HEADER-1X03 -> dn-electronics:HEADER-1X03
- SW1, SW2: device david-norman:SMT-SWITCH -> dn-electronics:SWITCH-2PIN
- U1: device david-norman:USB-A-PLUG-V1 -> dn-electronics:USB-TYPEA-PLUG
Connections:
- net GND: now also JP2.3; no longer JP1.GND
- net N$11: now also IC1.PC1(RESET), JP2.1; no longer IC1.PC1(/RESET), JP1.RESET
- net N$12: now also JP1.3; no longer JP2.3
- net N$5: now also JP1.1; no longer JP2.1
- net N$6: now also JP1.2; no longer JP2.2
- net N$9: now also JP2.2; no longer JP1.HWB
Other:
- moved on the sheet: C1, C2, C3, C4, C5, C6, C7, C8, D1, IC1, IR1, JP2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
